File: flipdotUSV.kicad_pcb (KiCad board)
At the start: 2 copper layers, 65 x 56.5 mm, 26 parts, among them IC1 ATTINY85-P, P2 CONN_01X02, P3 Raspberry_Pi_+_Conn, P4 CONN_01X02, Q1 BC547, U1 LM2596S-5

Commit message: add Layout
Parts:
- added C4: 10n, Capacitors_SMD:C_0805_HandSoldering, F.Cu at (151.3, 99.0)
- added C5: 100n, Capacitors_SMD:C_0805_HandSoldering, F.Cu at (154.1, 99.0)
- added C6: DNL, Capacitors_SMD:CP_Elec_10x10, F.Cu at (124.1, 88.7)
- added C7: 100nF, Capacitors_SMD:C_0805_HandSoldering, F.Cu at (121.8, 96.7)
- added G***: LOGO, flipdot:logo_15x15, F.Cu at (110.7, 87.6)
- added R8: 330k, Resistors_SMD:R_0805_HandSoldering, F.Cu at (122.1, 105.1)
- added R9: 100k, Resistors_SMD:R_0805_HandSoldering, F.Cu at (116.3, 96.8)
- added RL1: HFD2-L2, HFD2-L2:HFD2-L2, F.Cu at (141.3, 110.5)
- C1: footprint Capacitors_SMD:C_0805_HandSoldering -> Capacitors_SMD:CP_Elec_10x10
- C2: value 680uF -> 1mF; footprint Capacitors_SMD:c_elec_4x5.8 -> Capacitors_SMD:CP_Elec_10x10
- C3: value 220uF -> 1mF; footprint Capacitors_SMD:c_elec_4x5.8 -> Capacitors_SMD:CP_Elec_10x10
- D1, D2, D3, D5: footprint Diodes_SMD:MiniMELF_Handsoldering -> Diodes_SMD:D_SMA_Handsoldering
- D4: footprint Diodes_SMD:MiniMELF_Handsoldering -> Diodes_SMD:D_SMB-SMC_Universal_Handsoldering
- IC1: value ATTINY85-P -> ATTINY13-S; footprint Housings_DIP:DIP-8_W7.62mm_LongPads -> SMD_Packages:SOIC-8-N
- L1: footprint Inductors:SELF-WE-PD-XXL -> Choke_SMD:Choke_SMD_12x12mm_h8mm
- P2, P4: footprint Connect:PINHEAD1-2 -> smd_proto:AK300-2_without
- P3: footprint Connect:IDC_Header_Straight_40pins -> smd_proto:IDC_Header_Straight_40pins_without
- R1, R3, R4, R5: moved to F.Cu
- R2: footprint Resistors_SMD:R_0805_HandSoldering -> Resistors_ThroughHole:R_Axial_Power_L25.0mm_W6.4mm_P30.48mm; moved to F.Cu
- moved D3 95.4 mm to (155.1, 114.2), turned to 270 degrees
- moved R2 77.6 mm to (160.6, 122.7), turned to 180 degrees
- moved P4 56.9 mm to (110.2, 117.1)
- moved R3 51.9 mm to (115.3, 123.5), turned to 90 degrees
- moved L1 50.3 mm to (149.1, 88.7), turned to 90 degrees
- moved C3 48.9 mm to (136.1, 88.7), turned to 90 degrees
- moved D4 43.2 mm to (162.9, 102.7)
- moved R7 40.8 mm to (128.6, 97.8)
- moved IC1 40.2 mm to (122.1, 100.5), turned to 270 degrees
- moved D5 39.0 mm to (147.5, 99.9), turned to 270 degrees
- moved D1 38.2 mm to (143.6, 100.0), turned to 270 degrees
- moved R6 36.5 mm to (133.2, 101.3), turned to 270 degrees
- moved Q1 35.3 mm to (138.1, 101.7)
- moved R1 32.6 mm to (117.8, 123.5), turned to 90 degrees
- moved C1 32.4 mm to (123.7, 114.6), turned to 90 degrees
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Connections:
- IC1 pad 3: (no net) -> Voltage
- P3 pad 11: (no net) -> RPI_READBACK
- P3 pad 13: (no net) -> RPI_SHUTDOWN
- P3 pad 29: RPI_SHUTDOWN -> (no net)
- P3 pad 31: RPI_READBACK -> (no net)
- R2 pad 1: Net-(D2-Pad1) -> +BATT
- R2 pad 2: +BATT -> Net-(D2-Pad1)
- R3 pad 1: (no net) -> +14V
Routing:
- net +5V: track 3.03 -> 94.7 mm, vias 0 -> 2
- net +BATT: track 0.00 -> 74.9 mm
- net GND: track 74.4 -> 132.8 mm, vias 0 -> 9
- net Net-(D5-Pad2): track 0.00 -> 54.5 mm, vias 0 -> 2
- net Net-(D2-Pad1): track 0.00 -> 37.0 mm
- net Net-(C2-Pad1): track 0.00 -> 33.5 mm
- net RPI_SHUTDOWN: track 0.11 -> 33.1 mm, vias 0 -> 2
- net Net-(D4-Pad1): track 0.00 -> 29.9 mm, vias 0 -> 2
- net Batt_Voltage: track 0.00 -> 27.9 mm, vias 0 -> 1
- net RPI_READBACK: track 0.00 -> 27.3 mm
- net +14V: track 0.00 -> 26.2 mm
- net Net-(C1-Pad2): track 0.00 -> 24.3 mm
- net Rel_off: track 0.54 -> 19.9 mm
- net Voltage: track 0.00 -> 11.0 mm
- net Net-(Q1-Pad2): track 0.00 -> 9.13 mm, vias 0 -> 1
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- added copper zone on F.Cu, net +5V
Other:
- outline, holes or cut-outs redrawn
- board text added: "14V"
- board text added: "BAT"
- board text removed: "CERN OHL V1.2"
- board text removed: "Julien M."

Commit message: fixed footprint fuckup
Parts:
- P2, P4: footprint smd_proto:AK300-2_without -> Connect:AK300-2; moved to B.Cu
- P3: footprint smd_proto:IDC_Header_Straight_40pins_without -> Connect:IDC_Header_Straight_40pins
Routing:
- net +5V: track 94.7 -> 113.8 mm, vias 2 -> 3
- net +BATT: track 74.9 -> 60.1 mm
- net Net-(D2-Pad1): track 37.0 -> 44.5 mm
- net Rel_off: track 19.9 -> 13.2 mm
- net GND: track 132.8 -> 137.1 mm
- net Batt_Voltage: track 27.9 -> 32.1 mm, vias 1 -> 2
- net Net-(C2-Pad1): track 33.5 -> 30.1 mm
- net Net-(C1-Pad2): track 24.3 -> 25.9 mm

Commit message: add isp port
Parts:
- added CON1: AVR-ISP-6, Connect:IDC_Header_Straight_6pins, F.Cu at (109.5, 86.0)
- G***: moved to B.Cu
- IC1: footprint SMD_Packages:SOIC-8-N -> Housings_SOIC:SOIJ-8_5.3x5.3mm_Pitch1.27mm
- P2, P4: footprint Connect:AK300-2 -> HFD2-L2:AK300-2_my
- moved G*** 48.3 mm to (144.3, 122.3), turned to 180 degrees
- moved R9 8.52 mm to (117.4, 105.3), turned to 180 degrees
- moved P2 2.00 mm to (108.2, 106.7)
- moved P4 2.00 mm to (108.2, 117.1)
- moved IC1 0.67 mm to (121.4, 100.4), turned to 0 degrees
- moved R8 0.39 mm to (122.5, 105.3)
Connections:
- net Net-(D5-Pad2) renamed mosi
- net Net-(IC1-Pad6) renamed miso
- net Net-(IC1-Pad7) renamed sck
- IC1 pad 1: (no net) -> RST
Routing:
- net miso: track 2.37 -> 28.4 mm, vias 0 -> 1
- net sck: track 2.93 -> 26.9 mm, vias 0 -> 2
- net mosi: track 54.5 -> 75.8 mm
- net GND: track 137.1 -> 151.9 mm, vias 9 -> 7
- net RST: track 0.00 -> 12.6 mm
- net +5V: track 113.8 -> 103.1 mm, vias 3 -> 4
- net +BATT: track 60.1 -> 62.1 mm
- net Voltage: track 11.0 -> 9.21 mm
- net RPI_READBACK: track 27.3 -> 28.6 mm
- net (no net): track 0.54 -> 0.00 mm
